Commit message: manual_qr completed

File: mazix_description/urdf/lidar.urdf.xacro (robot description, xacro)
@@ -4,5 +4,5 @@
         <parent link="chassis"/>
         <child link="laser_frame"/>
-        <origin xyz="0.37 0 0.22" rpy="0 0 0"/>
+        <origin xyz="0.37 0 0.22" rpy="0 0 -${pi/2}"/>
     </joint>
     <link name="laser_frame">
@@ -27,16 +27,17 @@
             <pose> 0 0 0 0 0 0 </pose>
             <visualize>true</visualize>
-            <update_rate>10</update_rate>
+            <update_rate>15.0</update_rate>
             <ray>
                 <scan>
                     <horizontal>
                         <samples>360</samples>
-                        <min_angle>-3.14</min_angle>
-                        <max_angle>3.14</max_angle>
+                        <resolution>1</resolution>   <!-- degrees per point -->
+                        <min_angle>0.0</min_angle>
+                        <max_angle>3.14/2</max_angle>
                     </horizontal>
                 </scan>
                 <range>
-                    <min>0.3</min>
-                    <max>12</max>
+                    <min>0.1</min>
+                    <max>1</max>
                 </range>
             </ray>

Commit message: commit...

File: mazix_description/urdf/lidar.urdf.xacro (robot description, xacro)
@@ -39,5 +39,5 @@
                 <range>
                     <min>0.1</min>
-                    <max>1</max>
+                    <max>2</max>
                 </range>
             </ray>

File: mazix_description/urdf/robot_core.urdf.xacro (robot description, xacro)
@@ -35,5 +35,5 @@
             <origin xyz="0.135 0 0.052885"/>
             <geometry>
-                <box size="0.7 0.5 0.3"/>
+                <box size="0.5 0.4 0.3"/>
             </geometry>
             <material name="black"/>
@@ -42,5 +42,5 @@
             <origin xyz="0.135 0 0.052885"/>
             <geometry>
-                <box size="0.7 0.5 0.3"/>
+                <box size="0.5 0.4 0.3"/>
             </geometry>
         </collision>
@@ -56,5 +56,5 @@
         <parent link="base_link"/>
         <child link="left_wheel"/>
-        <origin xyz="-0.22 0.2 -0.15" rpy="-${pi/2} 0 0"/>  <!-- we are rotating the whole bot 90 degrees wrt x axis..-->
+        <origin xyz="0 0.15 -0.15" rpy="-${pi/2} 0 0"/>  <!-- we are rotating the whole bot 90 degrees wrt x axis..-->
         <axis xyz="0 0 1"/>
     </joint>
@@ -62,5 +62,5 @@
         <visual>
             <geometry>
-                <cylinder radius="0.08" length="0.070"/>
+                <cylinder radius="0.07" length="0.070"/>
             </geometry>
             <material name="white"/>
@@ -68,8 +68,8 @@
         <collision>
             <geometry>
-                <sphere radius="0.08"/>
+                <sphere radius="0.07"/>
             </geometry>
         </collision>
-        <xacro:inertial_cylinder mass="4" length="0.07" radius="0.08">
+        <xacro:inertial_cylinder mass="4" length="0.07" radius="0.07">
             <origin xyz = "0 0 0" rpy = "0 0 0 "/>
         </xacro:inertial_cylinder>
@@ -82,5 +82,5 @@
         <parent link="base_link"/>
         <child link="right_wheel"/>
-        <origin xyz="-0.22 -0.2 -0.15" rpy="${pi/2} 0 0"/>  <!-- we are rotating the whole bot 90 degrees wrt x axis..-->
+        <origin xyz="0 -0.15 -0.15" rpy="${pi/2} 0 0"/>  <!-- we are rotating the whole bot 90 degrees wrt x axis..-->
         <axis xyz="0 0 -1"/>
     </joint>
@@ -88,5 +88,5 @@
         <visual>
             <geometry>
-                <cylinder radius="0.08" length="0.070"/>
+                <cylinder radius="0.07" length="0.070"/>
             </geometry>
             <material name="white"/>
@@ -94,9 +94,9 @@
         <collision>
             <geometry>
-                <sphere radius="0.08"/>
+                <sphere radius="0.07"/>
             </geometry>
             <material name="white"/>
         </collision>
-        <xacro:inertial_cylinder mass="4" length="0.07" radius="0.08">
+        <xacro:inertial_cylinder mass="4" length="0.07" radius="0.07">
             <origin xyz = "0 0 0" rpy = "0 0 0 "/>
         </xacro:inertial_cylinder>
@@ -114,5 +114,5 @@
         <visual>
             <geometry>
-                <sphere radius="0.08"/>
+                <sphere radius="0.07"/>
             </geometry>
             <material name="white"/>
@@ -120,9 +120,9 @@
         <collision>
             <geometry>
-                <sphere radius="0.08"/>
+                <sphere radius="0.07"/>
             </geometry>
             <material name="white"/>
         </collision>
-        <xacro:inertial_sphere mass="5" radius="0.2">
+        <xacro:inertial_sphere mass="5" radius="0.07">
             <origin xyz="0 0 0" rpy="0 0 0"/>
         </xacro:inertial_sphere>
